Commit message: Gazebo simulation

File: catkin_ws/src/simulation/rm_description/urdf/links_joints.xacro (robot description, xacro)
@@ -1,4 +1,5 @@
 <?xml version="1.0"?>
 <robot xmlns:xacro="http://www.ros.org/wiki/xacro">
+    <!-- We need Inertia and Collision properties for Gazebo simulation -->
     <!-- Creating m_joint function for joints-->
     <xacro:macro name="m_joint" params="name type axis_xyz origin_rpy origin_xyz parent child">
@@ -12,6 +13,19 @@
     </xacro:macro>
     <!-- Creating m_link_cylinder function for links-->
-    <xacro:macro name="m_link_cylinder" params="name origin_rpy origin_xyz radius length">
+    <xacro:macro name="m_link_cylinder" params="name origin_rpy origin_xyz radius length mass ixx ixy ixz iyy iyz izz">
         <link name="${name}">
+            <!-- START Gazebo simulation properties -->
+            <inertial>
+                <mass value="${mass}"/>
+                <origin rpy="${origin_rpy}" xyz="${origin_xyz}"/>
+                <inertia ixx="${ixx}" ixy="${ixy}" ixz="${ixz}" iyy="${iyy}" iyz="${iyz}" izz="${izz}"/>
+            </inertial>
+            <collision>
+                <origin rpy="${origin_rpy}" xyz="${origin_xyz}"/>
+                <geometry>
+                    <cylinder radius="${radius}" length="${length}"/>
+                </geometry>
+            </collision>
+            <!-- END START Gazebo simulation properties -->
             <visual>
                 <origin rpy="${origin_rpy}" xyz="${origin_xyz}"/>
@@ -23,6 +37,19 @@
     </xacro:macro>
     <!-- Creating m_link_box function for link box-->
-    <xacro:macro name="m_link_box" params="name origin_rpy origin_xyz box_size">
+    <xacro:macro name="m_link_box" params="name origin_rpy origin_xyz box_size mass ixx ixy ixz iyy iyz izz">
         <link name="${name}">
+            <!-- START Gazebo simulation properties -->
+            <inertial>
+                <mass value="${mass}"/>
+                <origin rpy="${origin_rpy}" xyz="${origin_xyz}"/>
+                <inertia ixx="${ixx}" ixy="${ixy}" ixz="${ixz}" iyy="${iyy}" iyz="${iyz}" izz="${izz}"/>
+            </inertial>
+            <collision>
+                <origin rpy="${origin_rpy}" xyz="${origin_xyz}"/>
+                <geometry>
+                    <box size="${box_size}"/>
+                </geometry>
+            </collision>
+            <!-- END START Gazebo simulation properties -->
             <visual>
                 <origin rpy="${origin_rpy}" xyz="${origin_xyz}"/>

File: catkin_ws/src/simulation/rm_description/urdf/rm.xacro (robot description, xacro)
@@ -5,5 +5,7 @@
     <xacro:include filename="$(find rm_description)/urdf/robot_parameters.xacro"/>
     <!-- Base link box robot description-->
-    <m_link_box name="${l00}" origin_rpy="0 0 0" origin_xyz="0 0 0" box_size="1 1 1"/>
+    <m_link_box name="${l00}" origin_rpy="0 0 0" origin_xyz="0 0 0"
+                mass="1024" ixx="170.667" ixy="0" ixz="0" iyy="170.667" iyz="0" izz="170.667"
+                box_size="1 1 1"/>
 <!--    <link name="base_link">-->
 <!--        <visual>-->
@@ -29,5 +31,6 @@
     <!-- Link 1-->
     <m_link_cylinder name="${l01}" origin_rpy="0 0 0" origin_xyz="0 0 0.2"
-    radius="0.35" length="0.4"/>
+                     mass="157.633" ixx="13.235" ixy="0" ixz="0" iyy="13.235" iyz="0" izz="9.655"
+                     radius="0.35" length="0.4"/>
 <!--    <link name="link_01">-->
 <!--        <visual>S-->
@@ -51,5 +54,6 @@
     <!-- Link 2-->
     <m_link_cylinder name="${l02}" origin_rpy="0 0 0" origin_xyz="0 0 0.4"
-    radius="0.15" length="0.8"/>
+                     mass="57.906" ixx="12.679" ixy="0" ixz="0" iyy="12.679" iyz="0" izz="0.651"
+                     radius="0.15" length="0.8"/>
 <!--    <link name="link_02">-->
 <!--        <visual>-->
@@ -73,5 +77,6 @@
     <!-- Link 3-->
     <m_link_cylinder name="${l03}" origin_rpy="0 0 0" origin_xyz="0 0 0.4"
-    radius="0.15" length="0.8"/>
+                     mass="57.906" ixx="12.679" ixy="0" ixz="0" iyy="12.679" iyz="0" izz="0.651"
+                     radius="0.15" length="0.8"/>
 <!--    <link name="link_03">-->
 <!--        <visual>-->
@@ -95,5 +100,6 @@
     <!-- Link 4-->
     <m_link_cylinder name="${l04}" origin_rpy="0 0 0" origin_xyz="0 0 0.4"
-    radius="0.15" length="0.8"/>
+                     mass="57.906" ixx="12.679" ixy="0" ixz="0" iyy="12.679" iyz="0" izz="0.651"
+                     radius="0.15" length="0.8"/>
 <!--    <link name="link_04">-->
 <!--        <visual>-->
@@ -115,7 +121,8 @@
 <!--        <child link="link_05"/>-->
 <!--    </joint>-->
-    <!-- Link 5-->
+    <!-- Link 5 / End effector -->
     <m_link_cylinder name="${l05}" origin_rpy="0 0 0" origin_xyz="0 0 0.125"
-    radius="0.15" length="0.25"/>
+                     mass="18.056" ixx="0.479" ixy="0" ixz="0" iyy="0.479" iyz="0" izz="0.204"
+                     radius="0.15" length="0.25"/>
 <!--    <link name="link_05">-->
 <!--        <visual>-->
