Commit message: URDF xacro parameters

File: catkin_ws/src/simulation/rm_description/urdf/rm.xacro (robot description, xacro)
@@ -1,99 +1,128 @@
 <?xml version="1.0" ?>
 <robot name="rm" xmlns:xacro="http://www.ros.org/wiki/xacro">
-    <!-- Base link -->
-    <link name="base_link">
-        <visual>
-            <!-- Origin of the box -->
-            <origin rpy="0 0 0" xyz="0 0 0"/>
-            <geometry>
-                <!-- Box size in meters -->
-                <box size="1 1 1"/>
-            </geometry>
-        </visual>
-    </link>
+    <!-- Include the file to use the functions -->
+    <xacro:include filename="$(find rm_description)/urdf/links_joints.xacro"/>
+    <xacro:include filename="$(find rm_description)/urdf/robot_parameters.xacro"/>
+    <!-- Base link box robot description-->
+    <m_link_box name="${l00}" origin_rpy="0 0 0" origin_xyz="0 0 0" box_size="1 1 1"/>
+<!--    <link name="base_link">-->
+<!--        <visual>-->
+<!--            &lt;!&ndash; Origin of the box &ndash;&gt;-->
+<!--            <origin rpy="0 0 0" xyz="0 0 0"/>-->
+<!--            <geometry>-->
+<!--                &lt;!&ndash; Box size in meters &ndash;&gt;-->
+<!--                <box size="1 1 1"/>-->
+<!--            </geometry>-->
+<!--        </visual>-->
+<!--    </link>-->
     <!-- The circle joint between base_link and link_01 rotating around the z-axis -->
-    <joint name="base_link__link_01" type="revolute">
-        <axis xyz="0 0 1"/>
-        <limit effort="1000.0" lower="-3.14" upper="3.14" velocity="0.5"/>
-        <origin rpy="0 0 0" xyz="0 0 0.5"/>
-        <parent link="base_link"/>
-        <child link="link_01"/>
-    </joint>
+    <m_joint name="${l00}__${l01}" type="revolute" axis_xyz="0 0 1"
+             origin_rpy="0 0 0" origin_xyz="0 0 0.5"
+             parent="${l00}" child="${l01}"/>
+<!--    <joint name="base_link__link_01" type="revolute">-->
+<!--        <axis xyz="0 0 1"/>-->
+<!--        <limit effort="1000.0" lower="-3.14" upper="3.14" velocity="0.5"/>-->
+<!--        <origin rpy="0 0 0" xyz="0 0 0.5"/>-->
+<!--        <parent link="base_link"/>-->
+<!--        <child link="link_01"/>-->
+<!--    </joint>-->
     <!-- Link 1-->
-    <link name="link_01">
-        <visual>
-            <origin rpy="0 0 0" xyz="0 0 0.2"/>
-            <geometry>
-                <cylinder radius="0.35" length="0.4"/>
-            </geometry>
-        </visual>
-    </link>
+    <m_link_cylinder name="${l01}" origin_rpy="0 0 0" origin_xyz="0 0 0.2"
+    radius="0.35" length="0.4"/>
+<!--    <link name="link_01">-->
+<!--        <visual>S-->
+<!--            <origin rpy="0 0 0" xyz="0 0 0.2"/>-->
+<!--            <geometry>-->
+<!--                <cylinder radius="0.35" length="0.4"/>-->
+<!--            </geometry>-->
+<!--        </visual>-->
+<!--    </link>-->
     <!-- The circle joint between link_01 and link_02 rotating around the z-axis -->
-    <joint name="link_01__link_02" type="revolute">
-        <axis xyz="0 1 0"/>
-        <limit effort="1000.0" lower="-3.14" upper="3.14" velocity="0.5"/>
-        <origin rpy="0 0 0" xyz="0 0 0.4"/>
-        <parent link="link_01"/>
-        <child link="link_02"/>
-    </joint>
+    <m_joint name="${l01}__${l02}" type="revolute" axis_xyz="0 1 0"
+             origin_rpy="0 0 0" origin_xyz="0 0 0.4"
+             parent="${l01}" child="${l02}"/>
+<!--    <joint name="link_01__link_02" type="revolute">-->
+<!--        <axis xyz="0 1 0"/>-->
+<!--        <limit effort="1000.0" lower="-3.14" upper="3.14" velocity="0.5"/>-->
+<!--        <origin rpy="0 0 0" xyz="0 0 0.4"/>-->
+<!--        <parent link="link_01"/>-->
+<!--        <child link="link_02"/>-->
+<!--    </joint>-->
     <!-- Link 2-->
-    <link name="link_02">
-        <visual>
-            <origin rpy="0 0 0" xyz="0 0 0.4"/>
-            <geometry>
-                <cylinder radius="0.15" length="0.8"/>
-            </geometry>
-        </visual>
-    </link>
+    <m_link_cylinder name="${l02}" origin_rpy="0 0 0" origin_xyz="0 0 0.4"
+    radius="0.15" length="0.8"/>
+<!--    <link name="link_02">-->
+<!--        <visual>-->
+<!--            <origin rpy="0 0 0" xyz="0 0 0.4"/>-->
+<!--            <geometry>-->
+<!--                <cylinder radius="0.15" length="0.8"/>-->
+<!--            </geometry>-->
+<!--        </visual>-->
+<!--    </link>-->
     <!-- The circle joint between link_02 and link_03 rotating around the z-axis -->
-    <joint name="link_02__link_03" type="revolute">
-        <axis xyz="0 1 0"/>
-        <limit effort="1000.0" lower="-3.14" upper="3.14" velocity="0.5"/>
-        <origin rpy="0 0 0" xyz="0 0 0.8"/>
-        <parent link="link_02"/>
-        <child link="link_03"/>
-    </joint>
+    <m_joint name="${l02}__${l03}" type="revolute" axis_xyz="0 1 0"
+             origin_rpy="0 0 0" origin_xyz="0 0 0.8"
+             parent="${l02}" child="${l03}"/>
+<!--    <joint name="link_02__link_03" type="revolute">-->
+<!--        <axis xyz="0 1 0"/>-->
+<!--        <limit effort="1000.0" lower="-3.14" upper="3.14" velocity="0.5"/>-->
+<!--        <origin rpy="0 0 0" xyz="0 0 0.8"/>-->
+<!--        <parent link="link_02"/>-->
+<!--        <child link="link_03"/>-->
+<!--    </joint>-->
     <!-- Link 3-->
-    <link name="link_03">
-        <visual>
-            <origin rpy="0 0 0" xyz="0 0 0.4"/>
-            <geometry>
-                <cylinder radius="0.15" length="0.8"/>
-            </geometry>
-        </visual>
-    </link>
+    <m_link_cylinder name="${l03}" origin_rpy="0 0 0" origin_xyz="0 0 0.4"
+    radius="0.15" length="0.8"/>
+<!--    <link name="link_03">-->
+<!--        <visual>-->
+<!--            <origin rpy="0 0 0" xyz="0 0 0.4"/>-->
+<!--            <geometry>-->
+<!--                <cylinder radius="0.15" length="0.8"/>-->
+<!--            </geometry>-->
+<!--        </visual>-->
+<!--    </link>-->
     <!-- The circle joint between link_03 and link_04 rotating around the z-axis -->
-    <joint name="link_03__link_04" type="revolute">
-        <axis xyz="0 1 0"/>
-        <limit effort="1000.0" lower="-3.14" upper="3.14" velocity="0.5"/>
-        <origin rpy="0 0 0" xyz="0 0 0.8"/>
-        <parent link="link_03"/>
-        <child link="link_04"/>
-    </joint>
+    <m_joint name="${l03}__${l04}" type="revolute" axis_xyz="0 1 0"
+             origin_rpy="0 0 0" origin_xyz="0 0 0.8"
+             parent="${l03}" child="${l04}"/>
+<!--    <joint name="link_03__link_04" type="revolute">-->
+<!--        <axis xyz="0 1 0"/>-->
+<!--        <limit effort="1000.0" lower="-3.14" upper="3.14" velocity="0.5"/>-->
+<!--        <origin rpy="0 0 0" xyz="0 0 0.8"/>-->
+<!--        <parent link="link_03"/>-->
+<!--        <child link="link_04"/>-->
+<!--    </joint>-->
     <!-- Link 4-->
-    <link name="link_04">
-        <visual>
-            <origin rpy="0 0 0" xyz="0 0 0.4"/>
-            <geometry>
-                <cylinder radius="0.15" length="0.8"/>
-            </geometry>
-        </visual>
-    </link>
+    <m_link_cylinder name="${l04}" origin_rpy="0 0 0" origin_xyz="0 0 0.4"
+    radius="0.15" length="0.8"/>
+<!--    <link name="link_04">-->
+<!--        <visual>-->
+<!--            <origin rpy="0 0 0" xyz="0 0 0.4"/>-->
+<!--            <geometry>-->
+<!--                <cylinder radius="0.15" length="0.8"/>-->
+<!--            </geometry>-->
+<!--        </visual>-->
+<!--    </link>-->
     <!-- The circle joint between link_04 and link_05 rotating around the z-axis -->
-    <joint name="link_04__link_05" type="revolute">
-        <axis xyz="0 1 0"/>
-        <limit effort="1000.0" lower="-3.14" upper="3.14" velocity="0.5"/>
-        <origin rpy="0 0 0" xyz="0 0 0.8"/>
-        <parent link="link_04"/>
-        <child link="link_05"/>
-    </joint>
+    <m_joint name="${l04}__${l05}" type="revolute" axis_xyz="0 0 1"
+             origin_rpy="0 0 0" origin_xyz="0 0 0.8"
+             parent="${l04}" child="${l05}"/>
+<!--    <joint name="link_04__link_05" type="revolute">-->
+<!--        <axis xyz="0 0 1"/>-->
+<!--        <limit effort="1000.0" lower="-3.14" upper="3.14" velocity="0.5"/>-->
+<!--        <origin rpy="0 0 0" xyz="0 0 0.8"/>-->
+<!--        <parent link="link_04"/>-->
+<!--        <child link="link_05"/>-->
+<!--    </joint>-->
     <!-- Link 5-->
-    <link name="link_05">
-        <visual>
-            <origin rpy="0 0 0" xyz="0 0 0.125"/>
-            <geometry>
-                <cylinder radius="0.15" length="0.25"/>
-            </geometry>
-        </visual>
-    </link>
+    <m_link_cylinder name="${l05}" origin_rpy="0 0 0" origin_xyz="0 0 0.125"
+    radius="0.15" length="0.25"/>
+<!--    <link name="link_05">-->
+<!--        <visual>-->
+<!--            <origin rpy="0 0 0" xyz="0 0 0.125"/>-->
+<!--            <geometry>-->
+<!--                <cylinder radius="0.15" length="0.25"/>-->
+<!--            </geometry>-->
+<!--        </visual>-->
+<!--    </link>-->
 </robot>

Commit message: Added transmissions, joint state publisher needs to be improved

File: catkin_ws/src/simulation/rm_description/urdf/rm.xacro (robot description, xacro)
@@ -1,11 +1,18 @@
 <?xml version="1.0" ?>
 <robot name="rm" xmlns:xacro="http://www.ros.org/wiki/xacro">
-    <!-- Include the file to use the functions -->
-    <xacro:include filename="$(find rm_description)/urdf/links_joints.xacro"/>
-    <xacro:include filename="$(find rm_description)/urdf/robot_parameters.xacro"/>
-    <!-- Base link box robot description-->
-    <m_link_box name="${l00}" origin_rpy="0 0 0" origin_xyz="0 0 0"
-                mass="1024" ixx="170.667" ixy="0" ixz="0" iyy="170.667" iyz="0" izz="170.667"
-                box_size="1 1 1"/>
+  <!-- BGN - Include -->
+  <!-- Include the file to use the functions -->
+  <xacro:include filename="$(find rm_description)/urdf/robot_parameters.xacro" />
+  <xacro:include filename="$(find rm_description)/urdf/links_joints.xacro" />
+  <!-- END - Include -->
+  <!-- BGN - Robot description -->
+  <!-- Base link box robot description-->
+  <m_link_box name="${l00}"
+              origin_rpy="0 0 0" origin_xyz="0 0 0"
+              mass="1024"
+              ixx="170.667" ixy="0" ixz="0"
+              iyy="170.667" iyz="0"
+              izz="170.667"
+              box_size="1 1 1" />
 <!--    <link name="base_link">-->
 <!--        <visual>-->
@@ -18,8 +25,20 @@
 <!--        </visual>-->
 <!--    </link>-->
-    <!-- The circle joint between base_link and link_01 rotating around the z-axis -->
-    <m_joint name="${l00}__${l01}" type="revolute" axis_xyz="0 0 1"
-             origin_rpy="0 0 0" origin_xyz="0 0 0.5"
-             parent="${l00}" child="${l01}"/>
+  <!-- The circle joint between base_link and link_01 rotating around the z-axis -->
+  <m_joint name="${l00}__${l01}" type="revolute"
+           axis_xyz="0 0 1"
+           origin_rpy="0 0 0" origin_xyz="0 0 0.5"
+           parent="${l00}" child="${l01}" />
+  <!-- To use the controllers, add a new element for each joint we want to control which is called transmission -->
+  <transmission name="trans_${l00}__${l01}">
+    <type>transmission_interface/SimpleTransmission</type>
+    <joint name="${l00}__${l01}">
+      <hardwareInterface>hardware_interface/EffortJointInterface</hardwareInterface>
+    </joint>
+    <actuator name="motor_${l00}__${l01}">
+      <hardwareInterface>hardware_interface/EffortJointInterface</hardwareInterface>
+      <mechanicalReduction>1</mechanicalReduction>
+    </actuator>
+  </transmission>
 <!--    <joint name="base_link__link_01" type="revolute">-->
 <!--        <axis xyz="0 0 1"/>-->
@@ -29,107 +48,72 @@
 <!--        <child link="link_01"/>-->
 <!--    </joint>-->
-    <!-- Link 1-->
-    <m_link_cylinder name="${l01}" origin_rpy="0 0 0" origin_xyz="0 0 0.2"
-                     mass="157.633" ixx="13.235" ixy="0" ixz="0" iyy="13.235" iyz="0" izz="9.655"
-                     radius="0.35" length="0.4"/>
-<!--    <link name="link_01">-->
-<!--        <visual>S-->
-<!--            <origin rpy="0 0 0" xyz="0 0 0.2"/>-->
-<!--            <geometry>-->
-<!--                <cylinder radius="0.35" length="0.4"/>-->
-<!--            </geometry>-->
-<!--        </visual>-->
-<!--    </link>-->
-    <!-- The circle joint between link_01 and link_02 rotating around the z-axis -->
-    <m_joint name="${l01}__${l02}" type="revolute" axis_xyz="0 1 0"
-             origin_rpy="0 0 0" origin_xyz="0 0 0.4"
-             parent="${l01}" child="${l02}"/>
-<!--    <joint name="link_01__link_02" type="revolute">-->
-<!--        <axis xyz="0 1 0"/>-->
-<!--        <limit effort="1000.0" lower="-3.14" upper="3.14" velocity="0.5"/>-->
-<!--        <origin rpy="0 0 0" xyz="0 0 0.4"/>-->
-<!--        <parent link="link_01"/>-->
-<!--        <child link="link_02"/>-->
-<!--    </joint>-->
-    <!-- Link 2-->
-    <m_link_cylinder name="${l02}" origin_rpy="0 0 0" origin_xyz="0 0 0.4"
-                     mass="57.906" ixx="12.679" ixy="0" ixz="0" iyy="12.679" iyz="0" izz="0.651"
-                     radius="0.15" length="0.8"/>
-<!--    <link name="link_02">-->
-<!--        <visual>-->
-<!--            <origin rpy="0 0 0" xyz="0 0 0.4"/>-->
-<!--            <geometry>-->
-<!--                <cylinder radius="0.15" length="0.8"/>-->
-<!--            </geometry>-->
-<!--        </visual>-->
-<!--    </link>-->
-    <!-- The circle joint between link_02 and link_03 rotating around the z-axis -->
-    <m_joint name="${l02}__${l03}" type="revolute" axis_xyz="0 1 0"
-             origin_rpy="0 0 0" origin_xyz="0 0 0.8"
-             parent="${l02}" child="${l03}"/>
-<!--    <joint name="link_02__link_03" type="revolute">-->
-<!--        <axis xyz="0 1 0"/>-->
-<!--        <limit effort="1000.0" lower="-3.14" upper="3.14" velocity="0.5"/>-->
-<!--        <origin rpy="0 0 0" xyz="0 0 0.8"/>-->
-<!--        <parent link="link_02"/>-->
-<!--        <child link="link_03"/>-->
-<!--    </joint>-->
-    <!-- Link 3-->
-    <m_link_cylinder name="${l03}" origin_rpy="0 0 0" origin_xyz="0 0 0.4"
-                     mass="57.906" ixx="12.679" ixy="0" ixz="0" iyy="12.679" iyz="0" izz="0.651"
-                     radius="0.15" length="0.8"/>
-<!--    <link name="link_03">-->
-<!--        <visual>-->
-<!--            <origin rpy="0 0 0" xyz="0 0 0.4"/>-->
-<!--            <geometry>-->
-<!--                <cylinder radius="0.15" length="0.8"/>-->
-<!--            </geometry>-->
-<!--        </visual>-->
-<!--    </link>-->
-    <!-- The circle joint between link_03 and link_04 rotating around the z-axis -->
-    <m_joint name="${l03}__${l04}" type="revolute" axis_xyz="0 1 0"
-             origin_rpy="0 0 0" origin_xyz="0 0 0.8"
-             parent="${l03}" child="${l04}"/>
-<!--    <joint name="link_03__link_04" type="revolute">-->
-<!--        <axis xyz="0 1 0"/>-->
-<!--        <limit effort="1000.0" lower="-3.14" upper="3.14" velocity="0.5"/>-->
-<!--        <origin rpy="0 0 0" xyz="0 0 0.8"/>-->
-<!--        <parent link="link_03"/>-->
-<!--        <child link="link_04"/>-->
-<!--    </joint>-->
-    <!-- Link 4-->
-    <m_link_cylinder name="${l04}" origin_rpy="0 0 0" origin_xyz="0 0 0.4"
-                     mass="57.906" ixx="12.679" ixy="0" ixz="0" iyy="12.679" iyz="0" izz="0.651"
-                     radius="0.15" length="0.8"/>
-<!--    <link name="link_04">-->
-<!--        <visual>-->
-<!--            <origin rpy="0 0 0" xyz="0 0 0.4"/>-->
-<!--            <geometry>-->
-<!--                <cylinder radius="0.15" length="0.8"/>-->
-<!--            </geometry>-->
-<!--        </visual>-->
-<!--    </link>-->
-    <!-- The circle joint between link_04 and link_05 rotating around the z-axis -->
-    <m_joint name="${l04}__${l05}" type="revolute" axis_xyz="0 0 1"
-             origin_rpy="0 0 0" origin_xyz="0 0 0.8"
-             parent="${l04}" child="${l05}"/>
-<!--    <joint name="link_04__link_05" type="revolute">-->
-<!--        <axis xyz="0 0 1"/>-->
-<!--        <limit effort="1000.0" lower="-3.14" upper="3.14" velocity="0.5"/>-->
-<!--        <origin rpy="0 0 0" xyz="0 0 0.8"/>-->
-<!--        <parent link="link_04"/>-->
-<!--        <child link="link_05"/>-->
-<!--    </joint>-->
-    <!-- Link 5 / End effector -->
-    <m_link_cylinder name="${l05}" origin_rpy="0 0 0" origin_xyz="0 0 0.125"
-                     mass="18.056" ixx="0.479" ixy="0" ixz="0" iyy="0.479" iyz="0" izz="0.204"
-                     radius="0.15" length="0.25"/>
-<!--    <link name="link_05">-->
-<!--        <visual>-->
-<!--            <origin rpy="0 0 0" xyz="0 0 0.125"/>-->
-<!--            <geometry>-->
-<!--                <cylinder radius="0.15" length="0.25"/>-->
-<!--            </geometry>-->
-<!--        </visual>-->
-<!--    </link>-->
+  <!-- Link 1-->
+  <m_link_cylinder name="${l01}"
+              origin_rpy="0 0 0" origin_xyz="0 0 0.2"
+              mass="157.633"
+              ixx="13.235" ixy="0" ixz="0"
+              iyy="13.235" iyz="0"
+              izz="9.655"
+              length="0.4" radius="0.35" />
+  <m_joint name="${l01}__${l02}" type="revolute"
+           axis_xyz="0 1 0"
+           origin_rpy="0 0 0" origin_xyz="0 0 0.4"
+           parent="${l01}" child="${l02}" />
+  <transmission name="trans_${l01}__${l02}">
+    <type>transmission_interface/SimpleTransmission</type>
+    <joint name="${l01}__${l02}">
+      <hardwareInterface>hardware_interface/EffortJointInterface</hardwareInterface>
+    </joint>
+    <actuator name="motor_${l01}__${l02}">
+      <hardwareInterface>hardware_interface/EffortJointInterface</hardwareInterface>
+      <mechanicalReduction>1</mechanicalReduction>
+    </actuator>
+  </transmission>
+  <m_link_cylinder name="${l02}"
+              origin_rpy="0 0 0" origin_xyz="0 0 0.4"
+              mass="57.906"
+              ixx="12.679" ixy="0" ixz="0"
+              iyy="12.679" iyz="0"
+              izz="0.651"
+              radius="0.15" length="0.8" />
+  <!--
+  <m_joint name="${link_02_name}__${link_03_name}" type="revolute"
+           axis_xyz="0 1 0"
+           origin_rpy="0 0 0" origin_xyz="0 0 0.8"
+           parent="link_02" child="link_03" />
+  <m_link_cylinder name="${link_03_name}"
+              origin_rpy="0 0 0" origin_xyz="0 0 0.4"
+              mass="57.906"
+              ixx="12.679" ixy="0" ixz="0"
+              iyy="12.679" iyz="0"
+              izz="0.651"
+              radius="0.15" length="0.8" />
+  <m_joint name="${link_03_name}__${link_04_name}" type="revolute"
+           axis_xyz="0 1 0"
+           origin_rpy="0 0 0" origin_xyz="0 0 0.8"
+           parent="link_03" child="link_04" />
+  <m_link_cylinder name="${link_04_name}"
+              origin_rpy="0 0 0" origin_xyz="0 0 0.4"
+              mass="57.906"
+              ixx="12.679" ixy="0" ixz="0"
+              iyy="12.679" iyz="0"
+              izz="0.651"
+              radius="0.15" length="0.8" />
+  <m_joint name="${link_04_name}__${link_05_name}" type="revolute"
+           axis_xyz="0 0 1"
+           origin_rpy="0 0 0" origin_xyz="0 0 0.8"
+           parent="link_04" child="link_05" />
+  <m_link_cylinder name="${link_05_name}"
+              origin_rpy="0 0 0" origin_xyz="0 0 0.125"
+              mass="18.056"
+              ixx="0.479" ixy="0" ixz="0"
+              iyy="0.479" iyz="0"
+              izz="0.204"
+              radius="0.15" length="0.25" />
+  -->
+  <!-- END - Robot description -->
+  <gazebo>
+    <plugin name="gazebo_ros_control" filename="libgazebo_ros_control.so">
+    </plugin>
+  </gazebo>
 </robot>
