Commit message: ROS controllers implement to all joints of the robotic manipulator

File: rm_description/urdf/links_joints.xacro (robot description, xacro)
@@ -3,12 +3,23 @@
     <!-- We need Inertia and Collision properties for Gazebo simulation -->
     <!-- Creating m_joint function for joints-->
-    <xacro:macro name="m_joint" params="name type axis_xyz origin_rpy origin_xyz parent child">
+    <xacro:macro name="m_joint" params="name type axis_xyz origin_rpy origin_xyz parent child limit_effort limit_lower_val limit_upper_val limit_vel">
         <joint name="${name}" type="${type}">
             <axis xyz="${axis_xyz}"/>
-            <limit effort="1000.0" lower="-3.14" upper="3.14" velocity="0.5"/>
+            <limit effort="${limit_effort}" lower="${limit_lower_val}" upper="${limit_upper_val}" velocity="${limit_vel}"/>
             <origin rpy="${origin_rpy}" xyz="${origin_xyz}"/>
             <parent link="${parent}"/>
             <child link="${child}"/>
         </joint>
+        <!-- To use the controllers, add a new element for each joint we want to control which is called transmission -->
+        <transmission name="trans_${name}">
+            <type>transmission_interface/SimpleTransmission</type>
+            <joint name="${name}">
+                <hardwareInterface>hardware_interface/EffortJointInterface</hardwareInterface>
+            </joint>
+            <actuator name="motor_${name}">
+                <hardwareInterface>hardware_interface/EffortJointInterface</hardwareInterface>
+                <mechanicalReduction>1</mechanicalReduction>
+            </actuator>
+         </transmission>
     </xacro:macro>
     <!-- Creating m_link_cylinder function for links-->

File: rm_description/urdf/rm.xacro (robot description, xacro)
@@ -29,7 +29,11 @@
            axis_xyz="0 0 1"
            origin_rpy="0 0 0" origin_xyz="0 0 0.5"
-           parent="${l00}" child="${l01}" />
+           parent="${l00}" child="${l01}"
+           limit_effort="1000"
+           limit_lower_val="-3.14"
+           limit_upper_val="3.14"
+           limit_vel="0.5" />
   <!-- To use the controllers, add a new element for each joint we want to control which is called transmission -->
-  <transmission name="trans_${l00}__${l01}">
+  <!-- <transmission name="trans_${l00}__${l01}">
     <type>transmission_interface/SimpleTransmission</type>
     <joint name="${l00}__${l01}">
@@ -40,5 +44,5 @@
       <mechanicalReduction>1</mechanicalReduction>
     </actuator>
-  </transmission>
+  </transmission> -->
 <!--    <joint name="base_link__link_01" type="revolute">-->
 <!--        <axis xyz="0 0 1"/>-->
@@ -59,6 +63,10 @@
            axis_xyz="0 1 0"
            origin_rpy="0 0 0" origin_xyz="0 0 0.4"
-           parent="${l01}" child="${l02}" />
-  <transmission name="trans_${l01}__${l02}">
+           parent="${l01}" child="${l02}"
+           limit_effort="1000"
+           limit_lower_val="0"
+           limit_upper_val="0.5"
+           limit_vel="0.5" />
+  <!-- <transmission name="trans_${l01}__${l02}">
     <type>transmission_interface/SimpleTransmission</type>
     <joint name="${l01}__${l02}">
@@ -69,5 +77,5 @@
       <mechanicalReduction>1</mechanicalReduction>
     </actuator>
-  </transmission>
+  </transmission> -->
   <m_link_cylinder name="${l02}"
               origin_rpy="0 0 0" origin_xyz="0 0 0.4"
@@ -77,10 +85,13 @@
               izz="0.651"
               radius="0.15" length="0.8" />
-  <!--
-  <m_joint name="${link_02_name}__${link_03_name}" type="revolute"
+  <m_joint name="${l02}__${l03}" type="revolute"
            axis_xyz="0 1 0"
            origin_rpy="0 0 0" origin_xyz="0 0 0.8"
-           parent="link_02" child="link_03" />
-  <m_link_cylinder name="${link_03_name}"
+           parent="link_02" child="link_03"
+           limit_effort="1000"
+           limit_lower_val="0"
+           limit_upper_val="0.75"
+           limit_vel="0.5" />
+  <m_link_cylinder name="${l03}"
               origin_rpy="0 0 0" origin_xyz="0 0 0.4"
               mass="57.906"
@@ -89,9 +100,13 @@
               izz="0.651"
               radius="0.15" length="0.8" />
-  <m_joint name="${link_03_name}__${link_04_name}" type="revolute"
+  <m_joint name="${l03}__${l04}" type="revolute"
            axis_xyz="0 1 0"
            origin_rpy="0 0 0" origin_xyz="0 0 0.8"
-           parent="link_03" child="link_04" />
-  <m_link_cylinder name="${link_04_name}"
+           parent="link_03" child="link_04"
+           limit_effort="1000"
+           limit_lower_val="0"
+           limit_upper_val="0.75"
+           limit_vel="0.5" />
+  <m_link_cylinder name="${l04}"
               origin_rpy="0 0 0" origin_xyz="0 0 0.4"
               mass="57.906"
@@ -100,9 +115,13 @@
               izz="0.651"
               radius="0.15" length="0.8" />
-  <m_joint name="${link_04_name}__${link_05_name}" type="revolute"
+  <m_joint name="${l04}__${l05}" type="revolute"
            axis_xyz="0 0 1"
            origin_rpy="0 0 0" origin_xyz="0 0 0.8"
-           parent="link_04" child="link_05" />
-  <m_link_cylinder name="${link_05_name}"
+           parent="link_04" child="link_05"
+           limit_effort="1000"
+           limit_lower_val="-3.14"
+           limit_upper_val="3.14"
+           limit_vel="0.5" />
+  <m_link_cylinder name="${l05}"
               origin_rpy="0 0 0" origin_xyz="0 0 0.125"
               mass="18.056"
@@ -111,5 +130,4 @@
               izz="0.204"
               radius="0.15" length="0.25" />
-  -->
   <!-- END - Robot description -->
   <gazebo>

Commit message: Added new worlds

File: rm_description/urdf/links_joints.xacro (robot description, xacro)
@@ -71,3 +71,28 @@
         </link>
     </xacro:macro>
+    <!-- Mesh links -->
+    <xacro:macro name="m_link_mesh" params="name origin_xyz origin_rpy meshfile meshscale mass ixx ixy ixz iyy iyz izz">
+        <link name="${name}">
+            <!-- START Gazebo simulation properties -->
+            <inertial>
+                <mass value="${mass}"/>
+                <origin rpy="${origin_rpy}" xyz="${origin_xyz}"/>
+                <inertia ixx="${ixx}" ixy="${ixy}" ixz="${ixz}" iyy="${iyy}" iyz="${iyz}" izz="${izz}"/>
+            </inertial>
+            <collision>
+                <origin rpy="${origin_rpy}" xyz="${origin_xyz}"/>
+                <geometry>
+                    <mesh filename="${meshfile}" scale="${meshscale}"/>
+                </geometry>
+            </collision>
+            <!-- END START Gazebo simulation properties -->
+            <visual>
+                <origin rpy="${origin_rpy}" xyz="${origin_xyz}"/>
+                <geometry>
+                    <mesh filename="${meshfile}" scale="${meshscale}"/>
+                </geometry>
+                <material name="light_black"/>
+            </visual>
+        </link>
+    </xacro:macro>
 </robot>

File: rm_description/urdf/rm.xacro (robot description, xacro)
@@ -25,5 +25,5 @@
            limit_vel="0.5" />
   <!-- Link 1-->
-  <m_link_cylinder name="${l01}"
+  <!-- <m_link_cylinder name="${l01}"
               origin_rpy="0 0 0" origin_xyz="0 0 0.2"
               mass="157.633"
@@ -31,5 +31,13 @@
               iyy="13.235" iyz="0"
               izz="9.655"
-              length="0.4" radius="0.35" />
+              length="0.4" radius="0.35" /> -->
+  <m_link_mesh name="${l01}"
+            origin_rpy="0 0 0" origin_xyz="0 0 -0.1"
+            mass="157.633"
+            ixx="13.235" ixy="0" ixz="0"
+            iyy="13.235" iyz="0"
+            izz="9.655"
+            meshfile="package://rm_description/meshes/Link1-v2.stl"
+            meshscale="0.001 0.001 0.001" />
   <m_joint name="${l01}__${l02}" type="revolute"
            axis_xyz="0 1 0"
